File: PCB/NinjapadV2.kicad_pcb (KiCad board)
At the start: 2 copper layers, 63 x 64 mm, 25 parts, among them SW1 SW_Push_45deg, SW2 SW_Push_45deg, SW3 SW_Push_45deg, SW4 SW_Push_45deg, SW5 SW_Push_45deg, SW6 SW_Push_45deg, SW7 RotaryEncoder_Switch, U1 0.91"

Commit message: Add files via upload
Parts:
- L1: renamed from D7; footprint LED_SMD:LED_SK6812MINI-E_3.2x2.8mm_P1.5mm_ReverseMount -> LED footprint:MX_SK6812MINI-E_REV; moved to F.Cu
- L2: renamed from D8; footprint LED_SMD:LED_SK6812MINI-E_3.2x2.8mm_P1.5mm_ReverseMount -> LED footprint:MX_SK6812MINI-E_REV; moved to F.Cu
- L3: renamed from D9; footprint LED_SMD:LED_SK6812MINI-E_3.2x2.8mm_P1.5mm_ReverseMount -> LED footprint:MX_SK6812MINI-E_REV; moved to F.Cu
- L4: renamed from D10; footprint LED_SMD:LED_SK6812MINI-E_3.2x2.8mm_P1.5mm_ReverseMount -> LED footprint:MX_SK6812MINI-E_REV; moved to F.Cu
- L5: renamed from D11; footprint LED_SMD:LED_SK6812MINI-E_3.2x2.8mm_P1.5mm_ReverseMount -> LED footprint:MX_SK6812MINI-E_REV; moved to F.Cu
- L6: renamed from D12; footprint LED_SMD:LED_SK6812MINI-E_3.2x2.8mm_P1.5mm_ReverseMount -> LED footprint:MX_SK6812MINI-E_REV; moved to F.Cu
- moved L3 4.56 mm to (115.0, 45.0), turned to 0 degrees
- moved L1 4.54 mm to (153.1, 45.0), turned to 0 degrees
- moved L2 4.54 mm to (134.1, 45.0), turned to 0 degrees
- moved L6 4.51 mm to (115.0, 64.0), turned to 0 degrees
- moved L4 4.49 mm to (153.1, 64.0), turned to 0 degrees
- moved L5 4.49 mm to (134.1, 64.0), turned to 0 degrees
- moved D1 0.38 mm to (107.0, 53.5)
- moved D2 0.38 mm to (126.0, 53.5)
- moved D3 0.38 mm to (145.0, 53.5)
Routing:
- net 3.3V: track 196.7 -> 199.6 mm
- net Net-(L3-DOUT): track 85.3 -> 87.7 mm
- net GND: track 211.4 -> 210.3 mm
- net row2: track 104.5 -> 105.5 mm
